File: rat_board.sch (KiCad schematic (older format))
At the start: 51 parts, among them P1 FRONT_LEFT_IR, P2 SIDE_LEFT_IR, P3 SIDE_RIGHT_IR, P4 FRONT_RIGHT_IR, P5 LEFT_MOTOR, P6 RIGHT_MOTOR, P7 JTAG, P8 CONN_01X02, P9 CONN_01X04, SW1 SW_PUSH_SMALL_H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

Commit message: releseable board
Parts:
- removed C10, C9: 20p, Capacitors_SMD:C_0603_HandSoldering, symbol C
- removed D3: LED_1, LEDs:LED-3MM, symbol LED
- removed D4: LED_2, LEDs:LED-3MM, symbol LED
- removed D5: LED_3, LEDs:LED-3MM, symbol LED
- removed D6: LED_4, LEDs:LED-3MM, symbol LED
- removed D7: LED_5, LEDs:LED-3MM, symbol LED
- removed P1: FRONT_LEFT_IR, Pin_Headers:Pin_Header_Straight_1x03, symbol CONN_01X03
- removed P2: SIDE_LEFT_IR, Pin_Headers:Pin_Header_Straight_1x03, symbol CONN_01X03
- removed P3: SIDE_RIGHT_IR, Pin_Headers:Pin_Header_Straight_1x03, symbol CONN_01X03
- removed P4: FRONT_RIGHT_IR, Pin_Headers:Pin_Header_Straight_1x03, symbol CONN_01X03
- removed P5: LEFT_MOTOR, Pin_Headers:Pin_Header_Straight_1x06, symbol CONN_01X06
- removed P6: RIGHT_MOTOR, Pin_Headers:Pin_Header_Straight_1x06, symbol CONN_01X06
- removed P7: JTAG, Pin_Headers:Pin_Header_Angled_1x04, symbol CONN_01X04
- removed P9: CONN_01X04, symbol CONN_01X04
- removed R11, R12, R3, R4, R5: 100, Resistors_SMD:R_0603_HandSoldering, symbol R
- removed SW2: SWITCH_INV, custom-lib:TR05S3V3, symbol SWITCH_INV
- removed SW3: SELECT_BUTTON, Buttons_Switches_ThroughHole:SW_PUSH_6mm, symbol SW_PUSH
- removed Y1: 32.768kHz, Crystals:Crystal_MC-156, symbol Crystal
- added J1: CONN_01X08, Socket_Strips:Socket_Strip_Angled_1x08, symbol CONN_01X08
- added P1, P2: CONN_01X02, Socket_Strips:Socket_Strip_Straight_1x02, symbol CONN_01X02
- added R13, R14, R15: 47, Resistors_SMD:R_0603_HandSoldering, symbol R
- added RN1, RN3: 47k, Resistors_SMD:R_Array_Convex_4x0603, symbol R_Pack04
- added U10, U11, U4, U5, U6, U7, U8, U9: QRE1113, custom-lib:QRE1113GR, symbol QRE1113
- D1: symbol LED -> LED-RESCUE-rat_board
- D2: footprint LEDs:LED-3MM -> LEDs:LED_0603; symbol LED -> LED-RESCUE-rat_board
- R7: value 10k -> 47
- U1: footprint Pin_Headers:Pin_Header_Angled_1x03 -> custom-lib:TR05S3V3
Connections:
- net labels added: IR0, IR5, IR6, IR7
- net labels removed: ENC1A, ENC1B, ENC2A, ENC2B, LED1, LED2, LED3, LED4, LED5, OSC32IN, OSC32OUT, UB_SELECT
- wire segments 194 -> 179
- no-connect marks 6 -> 13
Other:
- note added: "INFRARED ARRAY"
- note added: "MOTOR CONNECTORS"
- note added: "SERIAL CONNECTOR"
- note removed: "SENSOR / MOTOR CONNECTORS"
- moved on the sheet: C1, C11, C12, C13, C14, C7, C8, P8, R1, R10, R2, R6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
